Commit message: chore: commit all pending workspace changes

File: gbt_description/urdf/GBT_C5A.urdf (robot description, URDF)
Before this commit: robot gbt_description, 7 links, 6 joints
Links:
- link base_link: mass 1.11799442797851 -> 9.16039502558691; geometry collision mesh filename=package://gbt_description/meshes/collision/c5a/c5a_base.STL; visual mesh filename=package://gbt_description/meshes/visual/c5a/c5a_base.dae
- link link1: mass 2.04479035782127 -> 15.175; geometry collision mesh filename=package://gbt_description/meshes/collision/c5a/c5a_1.STL; visual mesh filename=package://gbt_description/meshes/visual/c5a/c5a_1.dae
- link link2: mass 6.10875492875952 -> 45.747; geometry collision mesh filename=package://gbt_description/meshes/collision/c5a/c5a_2.STL; visual mesh filename=package://gbt_description/meshes/visual/c5a/c5a_2.dae
- link link3: mass 3.27878276509859 -> 25.388; geometry collision mesh filename=package://gbt_description/meshes/collision/c5a/c5a_3.STL; visual mesh filename=package://gbt_description/meshes/visual/c5a/c5a_3.dae
- link link4: mass 0.804364163350571 -> 5.9625; geometry collision mesh filename=package://gbt_description/meshes/collision/c5a/c5a_4.STL; visual mesh filename=package://gbt_description/meshes/visual/c5a/c5a_4.dae
- link link5: mass 0.802210955732477 -> 6.3692; geometry collision mesh filename=package://gbt_description/meshes/collision/c5a/c5a_5.STL; visual mesh filename=package://gbt_description/meshes/visual/c5a/c5a_5.dae
- link link6: mass 0.129160189065118 -> 1.0139; geometry collision mesh filename=package://gbt_description/meshes/collision/c5a/c5a_6.STL; visual mesh filename=package://gbt_description/meshes/visual/c5a/c5a_6.dae
Joints:
- joint joint1: limit lower=-6.283185307179 upper=6.283185307179 effort=10.0 velocity=3.14159 -> lower=-6.283185307179 upper=6.283185307179 effort=100 velocity=1; origin xyz=0 0 0.094 rpy=0 0 -1.570797 -> xyz=0 0 0.094 rpy=0 0 0
- joint joint2: limit lower=-1.483529864195 upper=4.625122517784 effort=10.0 velocity=3.14159 -> lower=-1.483529864195 upper=4.625122517784 effort=100 velocity=1; origin xyz=0.0630000000000007 0 0.0840208674128905 rpy=1.57079632679489 -1.5707963267949 1.5707963267949 -> xyz=0 0.063 0.084 rpy=-1.5708 0 0
- joint joint3: limit lower=-2.80998009571 upper=2.80998009571 effort=10.0 velocity=3.14159 -> lower=-2.809980095710 upper=2.809980095710 effort=100 velocity=1; origin xyz=0 0.42497913258711 0.00599999999999846 rpy=-3.14159265358979 0 3.14159265358979 -> xyz=0.425 0 0 rpy=-3.1416 0 3.1416
- joint joint4: limit lower=-1.483529864195 upper=4.625122517784 effort=10.0 velocity=3.14159 -> lower=-1.483529864195 upper=4.625122517784 effort=100 velocity=1; origin xyz=0 0.385 0.00370000000000101 rpy=3.14159265358979 0 1.5707963267949 -> xyz=-0.385 0 -0.0083 rpy=-3.1416 0 3.1416
- joint joint5: limit lower=-6.283185307179 upper=6.283185307179 effort=10.0 velocity=3.14159 -> lower=-6.283185307179 upper=6.283185307179 effort=100 velocity=1; origin xyz=0 0.065299999999999 0.0579999999999997 rpy=1.5707963267949 -1.5707963267949 0 -> xyz=0 0.0713 0.052 rpy=1.5708 0 0
- joint joint6: limit lower=-6.283185307179 upper=6.283185307179 effort=10.0 velocity=3.14159 -> lower=-6.283185307179 upper=6.283185307179 effort=100 velocity=1; origin xyz=0.0652999999999996 0 -0.0580000000000009 rpy=-1.5707963267949 0 -1.5707963267949 -> xyz=0 0.0713 -0.052 rpy=-1.5708 0 0

File: gbt_description/urdf/GBT_C5A_gazebo.urdf (robot description, URDF)
Before this commit: robot gbt_description, 7 links, 6 joints
Links:
- link base_link: mass 1.11799442797851 -> 9.16039502558691; geometry collision mesh filename=file://$(find gbt_description)/meshes/collision/c5a/c5a_bas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; visual mesh filename=file://$(find gbt_description)/meshes/visual/c5a/c5a_base.d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
- link link1: mass 2.04479035782127 -> 15.175; geometry collision mesh filename=file://$(find gbt_description)/meshes/collision/c5a/c5a_1.S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; visual mesh filename=file://$(find gbt_description)/meshes/visual/c5a/c5a_1.dae
- link link2: mass 6.10875492875952 -> 45.747; geometry collision mesh filename=file://$(find gbt_description)/meshes/collision/c5a/c5a_2.S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; visual mesh filename=file://$(find gbt_description)/meshes/visual/c5a/c5a_2.dae
- link link3: mass 3.27878276509859 -> 25.388; geometry collision mesh filename=file://$(find gbt_description)/meshes/collision/c5a/c5a_3.S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; visual mesh filename=file://$(find gbt_description)/meshes/visual/c5a/c5a_3.dae
- link link4: mass 0.804364163350571 -> 5.9625; geometry collision mesh filename=file://$(find gbt_description)/meshes/collision/c5a/c5a_4.S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; visual mesh filename=file://$(find gbt_description)/meshes/visual/c5a/c5a_4.dae
- link link5: mass 0.802210955732477 -> 6.3692; geometry collision mesh filename=file://$(find gbt_description)/meshes/collision/c5a/c5a_5.S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; visual mesh filename=file://$(find gbt_description)/meshes/visual/c5a/c5a_5.dae
- link link6: mass 0.129160189065118 -> 1.0139; geometry collision mesh filename=file://$(find gbt_description)/meshes/collision/c5a/c5a_6.S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; visual mesh filename=file://$(find gbt_description)/meshes/visual/c5a/c5a_6.dae
Joints:
- joint joint1: limit lower=-6.283185307179 upper=6.283185307179 effort=10.0 velocity=3.14159 -> lower=-6.283185307179 upper=6.283185307179 effort=100 velocity=1; origin xyz=0 0 0.094 rpy=0 0 -1.570797 -> xyz=0 0 0.094 rpy=0 0 0
- joint joint2: limit lower=-1.483529864195 upper=4.625122517784 effort=10.0 velocity=3.14159 -> lower=-1.483529864195 upper=4.625122517784 effort=100 velocity=1; origin xyz=0.0630000000000007 0 0.0840208674128905 rpy=1.57079632679489 -1.5707963267949 1.5707963267949 -> xyz=0 0.063 0.084 rpy=-1.5708 0 0
- joint joint3: limit lower=-2.80998009571 upper=2.80998009571 effort=10.0 velocity=3.14159 -> lower=-2.809980095710 upper=2.809980095710 effort=100 velocity=1; origin xyz=0 0.42497913258711 0.00599999999999846 rpy=-3.14159265358979 0 3.14159265358979 -> xyz=0.425 0 0 rpy=-3.1416 0 3.1416
- joint joint4: limit lower=-1.483529864195 upper=4.625122517784 effort=10.0 velocity=3.14159 -> lower=-1.483529864195 upper=4.625122517784 effort=100 velocity=1; origin xyz=0 0.385 0.00370000000000101 rpy=3.14159265358979 0 1.5707963267949 -> xyz=-0.385 0 -0.0083 rpy=-3.1416 0 3.1416
- joint joint5: limit lower=-6.283185307179 upper=6.283185307179 effort=10.0 velocity=3.14159 -> lower=-6.283185307179 upper=6.283185307179 effort=100 velocity=1; origin xyz=0 0.065299999999999 0.0579999999999997 rpy=1.5707963267949 -1.5707963267949 0 -> xyz=0 0.0713 0.052 rpy=1.5708 0 0
- joint joint6: limit lower=-6.283185307179 upper=6.283185307179 effort=10.0 velocity=3.14159 -> lower=-6.283185307179 upper=6.283185307179 effort=100 velocity=1; origin xyz=0.0652999999999996 0 -0.0580000000000009 rpy=-1.5707963267949 0 -1.5707963267949 -> xyz=0 0.0713 -0.052 rpy=-1.5708 0 0

File: gbt_gazebo/config/gazebo_c5a_description.urdf.xacro (robot description, xacro)
@@ -1,5 +1,5 @@
 <?xml version="1.0"?>
 <robot xmlns:xacro="http://www.ros.org/wiki/xacro" name="c5a_description">
-    <!-- Used for fixing robot to Gazebo 'base_link' 将机械手的基座固定在世界坐标上-->
+    <!-- Used for fixing robot to Gazebo 'base_link' -->
     <link name="world"/>
     <joint name="fixed" type="fixed">
@@ -9,5 +9,5 @@
     <!-- Import c5a_description urdf file -->
     <xacro:include filename="$(find gbt_description)/urdf/GBT_C5A_gazebo.urdf" />
-    <!-- 对一些link进行gazebo的属性设置 -->
+    <!-- Set Gazebo properties for certain links. -->
     <gazebo reference="base_link">
         <self_collide>false</self_collide>
@@ -15,26 +15,26 @@
     </gazebo>
     <gazebo reference="link1">
-        <material>Gazebo/White</material>
+        <!-- <material>Gazebo/White</material> -->
         <self_collide>false</self_collide>
         <gravity>false</gravity>
     </gazebo>
     <gazebo reference="link2">
-        <material>Gazebo/Red</material>
+        <!-- <material>Gazebo/Red</material> -->
         <gravity>false</gravity>
     </gazebo>
     <gazebo reference="link3">
-        <material>Gazebo/Green</material>
+        <!-- <material>Gazebo/Green</material> -->
         <gravity>false</gravity>
     </gazebo>
     <gazebo reference="link4">
-        <material>azebo/Orange</material>
+        <!-- <material>azebo/Orange</material> -->
         <gravity>false</gravity>
     </gazebo>
     <gazebo reference="link5">
-        <material>Gazebo/Gray</material>
+        <!-- <material>Gazebo/Gray</material> -->
         <gravity>false</gravity>
     </gazebo>
     <gazebo reference="link6">
-        <material>Gazebo/Yellow</material>
+        <!-- <material>Gazebo/Yellow</material> -->
         <gravity>false</gravity>
     </gazebo>
@@ -43,5 +43,5 @@
         <self_collide>true</self_collide>
     </gazebo>
-    <!-- 声明ros2_control -->
+    <!-- ros2_control -->
     <ros2_control name="GazeboSystem" type="system">
         <hardware>
@@ -91,5 +91,5 @@
         </joint>
     </ros2_control>
-    <!-- 加载ros2_control插件 -->
+    <!-- load ros2_control plugin-->
     <gazebo>
         <plugin filename="libgazebo_ros2_control.so" name="gazebo_ros2_control">
